File: Electronica/Plataforma_soldadora.brd (EAGLE design)
At the start: 100.3 x 36.5 mm, 26 parts, among them J1 22-27-2021-02, SW2 ROTARTY_ENCODER, T1 BTA06400B, U1 RPDZN5W6H, U5 ESP32-C3_SUPERMINISMD

Commit message: Update
Parts:
- R5: value 4K7 -> 47K
Other:
- board text added: "XDeSIG 2548"
- board text removed: "XDeSIG 2544"
